File: COTS/COTS.brd (EAGLE design)
At the start: 76.2 x 79.7 mm, 9 parts

Commit message: Atualização
Parts:
- removed U$8: SWITCH_3PIN, CRD:SWITCH_3PIN_FOOTPRINT
- added SP2: AL11P, buzzer:AL11P
- added U$10: PRESSION_BUTTON, CRD:PRESSION_BUTTON_FOOTPRINT
- moved U$3 3.81 mm to (17.8, 36.8)
Connections:
- new net SIGNAL1: U$2.24, U$5.1
- net BUZZER: now also SP2.+; no longer U$5.1
- net GND: now also SP2.-
- net VIN: now also U$10.PL1, U$10.PR1; no longer U$8.PL2, U$8.PR2
- net V_BATTERY: now also U$10.PL2, U$10.PR2; no longer U$8.PL3, U$8.PR3
Routing:
- net SIGNAL1: track 0.00 -> 48.0 mm
- net VIN: track 68.1 -> 98.2 mm
- net BUZZER: track 53.8 -> 41.9 mm
- net SDA: track 102.7 -> 98.9 mm
- net 3V3: track 183.5 -> 179.7 mm
- net SCL: track 130.2 -> 130.9 mm
- net OPTOACOPLADOR2: track 28.4 -> 27.8 mm
