File: COTS/COTS.sch (EAGLE design)
At the start: 9 parts

Commit message: Atualização
Parts:
- removed U$8: SWITCH_3PIN, CRD:SWITCH_3PIN
- added SP2: AL11P, buzzer:AL11P
- added U$10: PRESSION_BUTTON, CRD:PRESSION_BUTTON
Connections:
- new net SIGNAL1: U$2.IO27, U$5.1
- net BUZZER: now also SP2.2; no longer U$5.1
- net GND: now also SP2.1
- net VIN: now also U$10.PL1, U$10.PR1; no longer U$8.PL2, U$8.PR2
- net V_BATTERY: now also U$10.PL2, U$10.PR2; no longer U$8.PL3, U$8.PR3
Other:
- note added: "Comunicação serial"
- note added: "Optoacopladores"
- note added: "Sinal e 3V3"
- note removed: "Buzzer e 3V3"

Commit message: feat: ajustes na placa em conexões
Other:
- note added: "A alimentação de 3.3v juntamente com o sinal do buzzer virá dessa placa"
- note added: "O sinal de ativação dos Skibs virá dessa placa dos pinos 12 e 13 do esp32"
- note added: "Utilizaremos as conexões de comunicação serial dessa placa"
- note added: "utilizaremos o conector de bateria e o GND dessa placa"
Changed lines of the file:
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@@
 <text x="145.796" y="8.636" size="1.778" layer="91">Comunicação serial</text>
 <text x="176.022" y="8.89" size="1.778" layer="91">Optoacopladores</text>
+<text x="83.82" y="119.38" size="1.778" layer="91">Utilizaremos as conexões de comunicação  serial dessa placa</text>
+<text x="83.82" y="114.3" size="1.778" layer="91">O sinal de ativação dos Skibs virá dessa placa dos pinos 12 e 13 do esp32</text>
+<text x="83.82" y="109.22" size="1.778" layer="91">A alimentação de 3.3v juntamente com o sinal do buzzer virá dessa placa</text>
+<text x="83.82" y="104.14" size="1.778" layer="91">utilizaremos o conector de bateria e o GND dessa placa</text>
 </plain>
 <instances>
