File: Placa de processamento/Placa de processamento.sch (EAGLE design)
At the start: 10 parts

Commit message: Placas
Parts:
- added U$10: JST2.54X2P, CRD:JST2.54X2P
Connections:
- removed net N$5: U$1.PR1
- removed net N$6: U$1.PL1
- new net RX0: U$10.1, U$9.IO3
- new net TX0: U$10.2, U$9.IO1
- net VIN: now also U$1.PL2, U$1.PR2; no longer U$1.PL3, U$1.PR3
- net V_BATTERY: now also U$1.PL1, U$1.PR1; no longer U$1.PL2, U$1.PR2
Changed lines of the file:
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@@
 <part name="U$9" library="ESP32-DEVKITV1" library_urn="urn:adsk.eagle:library:44018017" deviceset="ESP32DEVKITV1" device="" package3d_urn="urn:adsk.eagle:package:44018021/1"/>
 <part name="IC1" library="v-reg" library_urn="urn:adsk.eagle:library:409" deviceset="78XXL" device="" package3d_urn="urn:adsk.eagle:package:30361/1"/>
+<part name="U$10" library="CRD" library_urn="urn:adsk.eagle:library:39051337" deviceset="JST2.54X2P" device="" package3d_urn="urn:adsk.eagle:package:39191967/2"/>
 </parts>
 <sheets>
@@
 </plain>
 <instances>
-<instance part="U$1" gate="G$1" x="2.54" y="71.12" smashed="yes"/>
+<instance part="U$1" gate="G$1" x="17.78" y="71.12" smashed="yes"/>
 <instance part="U$2" gate="G$1" x="-35.56" y="7.62" smashed="yes"/>
 <instance part="U$3" gate="G$1" x="48.26" y="114.3" smashed="yes"/>
@@
 <attribute name="VALUE" x="157.48" y="63.5" size="1.778" layer="96"/>
 </instance>
+<instance part="U$10" gate="G$1" x="144.78" y="114.3" smashed="yes"/>
 </instances>
 <busses>
@@
 </segment>
 <segment>
+<pinref part="U$1" gate="G$1" pin="PL1"/>
+<wire x1="6.35" y1="58.42" x2="6.35" y2="48.26" width="0.1524" layer="91"/>
+<wire x1="6.35" y1="48.26" x2="7.62" y2="48.26" width="0.1524" layer="91"/>
+<label x="5.08" y="43.18" size="1.778" layer="95" rot="R90"/>
+</segment>
+<segment>
+<pinref part="U$1" gate="G$1" pin="PR1"/>
+<wire x1="6.35" y1="83.82" x2="6.35" y2="93.98" width="0.1524" layer="91"/>
+<wire x1="6.35" y1="93.98" x2="7.62" y2="93.98" width="0.1524" layer="91"/>
+<label x="5.08" y="88.9" size="1.778" layer="95" rot="R90"/>
+</segment>
+</net>
+<net name="VIN" class="0">
+<segment>
+<pinref part="U$9" gate="G$1" pin="VIN"/>
+<wire x1="40.64" y1="0" x2="33.02" y2="0" width="0.1524" layer="91"/>
+<label x="25.4" y="0" size="1.778" layer="95"/>
+</segment>
+<segment>
+<pinref part="IC1" gate="A" pin="IN"/>
+<wire x1="137.16" y1="73.66" x2="147.32" y2="73.66" width="0.1524" layer="91"/>
+<label x="137.16" y="73.66" size="1.778" layer="95"/>
+</segment>
+<segment>
+<pinref part="U$1" gate="G$1" pin="PL2"/>
+<wire x1="11.43" y1="58.42" x2="11.43" y2="48.26" width="0.1524" layer="91"/>
+<wire x1="11.43" y1="48.26" x2="12.7" y2="48.26" width="0.1524" layer="91"/>
+<label x="9.398" y="55.118" size="1.778" layer="95" rot="R270"/>
+</segment>
+<segment>
 <pinref part="U$1" gate="G$1" pin="PR2"/>
 <wire x1="11.43" y1="83.82" x2="11.43" y2="93.98" width="0.1524" layer="91"/>
@@
 <label x="11.176" y="87.122" size="1.778" layer="95" rot="R90"/>
 </segment>
-<segment>
-<pinref part="U$1" gate="G$1" pin="PL2"/>
-<wire x1="11.43" y1="58.42" x2="11.43" y2="48.26" width="0.1524" layer="91"/>
-<wire x1="11.43" y1="48.26" x2="12.7" y2="48.26" width="0.1524" layer="91"/>
-<label x="9.398" y="55.118" size="1.778" layer="95" rot="R270"/>
-</segment>
-</net>
-<net name="VIN" class="0">
-<segment>
-<pinref part="U$1" gate="G$1" pin="PR3"/>
-<wire x1="16.51" y1="83.82" x2="16.51" y2="93.98" width="0.1524" layer="91"/>
-<wire x1="16.51" y1="93.98" x2="17.78" y2="93.98" width="0.1524" layer="91"/>
-<label x="16.256" y="90.424" size="1.778" layer="95" rot="R90"/>
-</segment>
-<segment>
-<pinref part="U$1" gate="G$1" pin="PL3"/>
-<wire x1="16.51" y1="58.42" x2="16.51" y2="48.26" width="0.1524" layer="91"/>
-<wire x1="16.51" y1="48.26" x2="17.78" y2="48.26" width="0.1524" layer="91"/>
-<label x="16.51" y="48.006" size="1.778" layer="95" rot="R90"/>
-</segment>
-<segment>
-<pinref part="U$9" gate="G$1" pin="VIN"/>
-<wire x1="40.64" y1="0" x2="33.02" y2="0" width="0.1524" layer="91"/>
-<label x="25.4" y="0" size="1.778" layer="95"/>
-</segment>
-<segment>
-<pinref part="IC1" gate="A" pin="IN"/>
-<wire x1="137.16" y1="73.66" x2="147.32" y2="73.66" width="0.1524" layer="91"/>
-<label x="137.16" y="73.66" size="1.778" layer="95"/>
-</segment>
-</net>
-<net name="N$5" class="0">
-<segment>
-<pinref part="U$1" gate="G$1" pin="PR1"/>
-<wire x1="6.35" y1="83.82" x2="6.35" y2="93.98" width="0.1524" layer="91"/>
-<wire x1="6.35" y1="93.98" x2="7.62" y2="93.98" width="0.1524" layer="91"/>
-</segment>
-</net>
-<net name="N$6" class="0">
-<segment>
-<pinref part="U$1" gate="G$1" pin="PL1"/>
-<wire x1="6.35" y1="58.42" x2="6.35" y2="48.26" width="0.1524" layer="91"/>
-<wire x1="6.35" y1="48.26" x2="7.62" y2="48.26" width="0.1524" layer="91"/>
-</segment>
 </net>
 <net name="5V" class="0">
@@
 </segment>
 </net>
+<net name="RX0" class="0">
+<segment>
+<pinref part="U$10" gate="G$1" pin="1"/>
+<wire x1="142.24" y1="104.14" x2="142.24" y2="96.52" width="0.1524" layer="91"/>
+<label x="142.24" y="91.44" size="1.778" layer="95" rot="R90"/>
+</segment>
+<segment>
+<pinref part="U$9" gate="G$1" pin="IO3"/>
+<wire x1="76.2" y1="27.94" x2="83.82" y2="27.94" width="0.1524" layer="91"/>
+<label x="83.82" y="27.94" size="1.778" layer="95"/>
+</segment>
+</net>
+<net name="TX0" class="0">
+<segment>
+<pinref part="U$10" gate="G$1" pin="2"/>
+<wire x1="147.32" y1="104.14" x2="147.32" y2="96.52" width="0.1524" layer="91"/>
+<label x="147.32" y="91.44" size="1.778" layer="95" rot="R90"/>
+</segment>
+<segment>
+<pinref part="U$9" gate="G$1" pin="IO1"/>
+<wire x1="76.2" y1="30.48" x2="83.82" y2="30.48" width="0.1524" layer="91"/>
+<label x="83.82" y="30.48" size="1.778" layer="95"/>
+</segment>
+</net>

Commit message: Atualização
Parts:
- added SP1: AL11P, buzzer:AL11P
Connections:
- new net SIGNAL1: U$5.1, U$9.IO14
- net BUZZER: now also SP1.2, U$9.IO27; no longer U$5.1, U$9.IO14
- net GND: now also SP1.1
Other:
- note added: "Comunicação serial"
- note added: "Optoacopladores"
- note added: "Sinal e 3V3"
- note removed: "Sinais Buzzer e 3V3"
- note removed: "Sinais optoacplador"
Changed lines of the file:
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@@
 <part name="IC1" library="v-reg" library_urn="urn:adsk.eagle:library:409" deviceset="78XXL" device="" package3d_urn="urn:adsk.eagle:package:30361/1"/>
 <part name="U$10" library="CRD" library_urn="urn:adsk.eagle:library:39051337" deviceset="JST2.54X2P" device="" package3d_urn="urn:adsk.eagle:package:39191967/2"/>
+<part name="SP1" library="buzzer" library_urn="urn:adsk.eagle:library:113" deviceset="AL11P" device="" package3d_urn="urn:adsk.eagle:package:5308/1"/>
 </parts>
 <sheets>
@@
 <text x="42.672" y="120.904" size="1.778" layer="91">Battery 9V</text>
 <text x="59.944" y="120.904" size="1.778" layer="91">Sinais Skibs</text>
-<text x="77.216" y="120.904" size="1.778" layer="91">Sinais Buzzer e 3V3</text>
-<text x="106.68" y="120.904" size="1.778" layer="91">Sinais optoacplador</text>
+<text x="77.216" y="120.904" size="1.778" layer="91">Sinal e 3V3</text>
+<text x="106.68" y="120.904" size="1.778" layer="91">Optoacopladores</text>
+<text x="137.16" y="120.65" size="1.778" layer="91">Comunicação serial</text>
 </plain>
 <instances>
@@
 </instance>
 <instance part="U$10" gate="G$1" x="144.78" y="114.3" smashed="yes"/>
+<instance part="SP1" gate="G$1" x="180.34" y="114.3" smashed="yes">
+<attribute name="NAME" x="176.53" y="120.65" size="1.778" layer="95"/>
+<attribute name="VALUE" x="176.53" y="111.125" size="1.778" layer="96"/>
+</instance>
 </instances>
 <busses>
@@
 <label x="154.94" y="55.88" size="1.778" layer="95" rot="R90"/>
 </segment>
+<segment>
+<pinref part="SP1" gate="G$1" pin="1"/>
+<wire x1="175.26" y1="114.3" x2="172.72" y2="114.3" width="0.1524" layer="91"/>
+<wire x1="172.72" y1="114.3" x2="172.72" y2="106.68" width="0.1524" layer="91"/>
+<label x="172.72" y="106.68" size="1.778" layer="95"/>
+</segment>
 </net>
 <net name="TX1" class="0">
@@
 <net name="BUZZER" class="0">
 <segment>
+<pinref part="SP1" gate="G$1" pin="2"/>
+<wire x1="185.42" y1="114.3" x2="187.96" y2="114.3" width="0.1524" layer="91"/>
+<wire x1="187.96" y1="114.3" x2="187.96" y2="106.68" width="0.1524" layer="91"/>
+<label x="187.96" y="106.68" size="1.778" layer="95"/>
+</segment>
+<segment>
+<pinref part="U$9" gate="G$1" pin="IO27"/>
+<wire x1="40.64" y1="12.7" x2="33.02" y2="12.7" width="0.1524" layer="91"/>
+<label x="25.4" y="12.7" size="1.778" layer="95"/>
+</segment>
+</net>
+<net name="OPTOACOPLADOR1" class="0">
+<segment>
+<pinref part="U$6" gate="G$1" pin="1"/>
+<wire x1="111.76" y1="104.14" x2="111.76" y2="96.52" width="0.1524" layer="91"/>
+<label x="111.76" y="81.28" size="1.778" layer="95" rot="R90"/>
+</segment>
+<segment>
+<pinref part="U$9" gate="G$1" pin="IO34"/>
+<wire x1="40.64" y1="27.94" x2="33.02" y2="27.94" width="0.1524" layer="91"/>
+<label x="12.7" y="27.94" size="1.778" layer="95"/>
+</segment>
+</net>
+<net name="OPTOACOPLADOR2" class="0">
+<segment>
+<pinref part="U$6" gate="G$1" pin="2"/>
+<wire x1="116.84" y1="104.14" x2="116.84" y2="96.52" width="0.1524" layer="91"/>
+<label x="116.84" y="81.28" size="1.778" layer="95" rot="R90"/>
+</segment>
+<segment>
+<pinref part="U$9" gate="G$1" pin="IO35"/>
+<wire x1="40.64" y1="25.4" x2="33.02" y2="25.4" width="0.1524" layer="91"/>
+<label x="12.7" y="25.4" size="1.778" layer="95"/>
+</segment>
+</net>
+<net name="RX0" class="0">
+<segment>
+<pinref part="U$10" gate="G$1" pin="1"/>
+<wire x1="142.24" y1="104.14" x2="142.24" y2="96.52" width="0.1524" layer="91"/>
+<label x="142.24" y="91.44" size="1.778" layer="95" rot="R90"/>
+</segment>
+<segment>
+<pinref part="U$9" gate="G$1" pin="IO3"/>
+<wire x1="76.2" y1="27.94" x2="83.82" y2="27.94" width="0.1524" layer="91"/>
+<label x="83.82" y="27.94" size="1.778" layer="95"/>
+</segment>
+</net>
+<net name="TX0" class="0">
+<segment>
+<pinref part="U$10" gate="G$1" pin="2"/>
+<wire x1="147.32" y1="104.14" x2="147.32" y2="96.52" width="0.1524" layer="91"/>
+<label x="147.32" y="91.44" size="1.778" layer="95" rot="R90"/>
+</segment>
+<segment>
+<pinref part="U$9" gate="G$1" pin="IO1"/>
+<wire x1="76.2" y1="30.48" x2="83.82" y2="30.48" width="0.1524" layer="91"/>
+<label x="83.82" y="30.48" size="1.778" layer="95"/>
+</segment>
+</net>
+<net name="SIGNAL1" class="0">
+<segment>
+<pinref part="U$9" gate="G$1" pin="IO14"/>
+<wire x1="40.64" y1="10.16" x2="33.02" y2="10.16" width="0.1524" layer="91"/>
+<label x="25.4" y="10.16" size="1.778" layer="95"/>
+</segment>
+<segment>
 <pinref part="U$5" gate="G$1" pin="1"/>
 <wire x1="81.28" y1="104.14" x2="81.28" y2="96.52" width="0.1524" layer="91"/>
 <label x="81.28" y="88.9" size="1.778" layer="95" rot="R90"/>
 </segment>
-<segment>
-<pinref part="U$9" gate="G$1" pin="IO14"/>
-<wire x1="40.64" y1="10.16" x2="33.02" y2="10.16" width="0.1524" layer="91"/>
-<label x="25.4" y="10.16" size="1.778" layer="95"/>
-</segment>
-</net>
-<net name="OPTOACOPLADOR1" class="0">
-<segment>
-<pinref part="U$6" gate="G$1" pin="1"/>
-<wire x1="111.76" y1="104.14" x2="111.76" y2="96.52" width="0.1524" layer="91"/>
-<label x="111.76" y="81.28" size="1.778" layer="95" rot="R90"/>
-</segment>
-<segment>
-<pinref part="U$9" gate="G$1" pin="IO34"/>
-<wire x1="40.64" y1="27.94" x2="33.02" y2="27.94" width="0.1524" layer="91"/>
-<label x="12.7" y="27.94" size="1.778" layer="95"/>
-</segment>
-</net>
-<net name="OPTOACOPLADOR2" class="0">
-<segment>
-<pinref part="U$6" gate="G$1" pin="2"/>
-<wire x1="116.84" y1="104.14" x2="116.84" y2="96.52" width="0.1524" layer="91"/>
-<label x="116.84" y="81.28" size="1.778" layer="95" rot="R90"/>
-</segment>
-<segment>
-<pinref part="U$9" gate="G$1" pin="IO35"/>
-<wire x1="40.64" y1="25.4" x2="33.02" y2="25.4" width="0.1524" layer="91"/>
-<label x="12.7" y="25.4" size="1.778" layer="95"/>
-</segment>
-</net>
-<net name="RX0" class="0">
-<segment>
-<pinref part="U$10" gate="G$1" pin="1"/>
-<wire x1="142.24" y1="104.14" x2="142.24" y2="96.52" width="0.1524" layer="91"/>
-<label x="142.24" y="91.44" size="1.778" layer="95" rot="R90"/>
-</segment>
-<segment>
-<pinref part="U$9" gate="G$1" pin="IO3"/>
-<wire x1="76.2" y1="27.94" x2="83.82" y2="27.94" width="0.1524" layer="91"/>
-<label x="83.82" y="27.94" size="1.778" layer="95"/>
-</segment>
-</net>
-<net name="TX0" class="0">
-<segment>
-<pinref part="U$10" gate="G$1" pin="2"/>
-<wire x1="147.32" y1="104.14" x2="147.32" y2="96.52" width="0.1524" layer="91"/>
-<label x="147.32" y="91.44" size="1.778" layer="95" rot="R90"/>
-</segment>
-<segment>
-<pinref part="U$9" gate="G$1" pin="IO1"/>
-<wire x1="76.2" y1="30.48" x2="83.82" y2="30.48" width="0.1524" layer="91"/>
-<label x="83.82" y="30.48" size="1.778" layer="95"/>
-</segment>
-</net>
+</net>

Commit message: feat: ajustes na placa em conexões
Other:
- note added: "Seram utilizados os pinos 34 e 35 para os Octocopladores, utilizaremos a conexão de jst de optocopladores dessa placa para isso."
- note added: "Será utilizado as conexões seriais, dessa placa"
- note added: "Utilizaremos o conector de GND e Bateria dessa placa"
Changed lines of the file:
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@@
 <text x="106.68" y="120.904" size="1.778" layer="91">Optoacopladores</text>
 <text x="137.16" y="120.65" size="1.778" layer="91">Comunicação serial</text>
+<text x="38.1" y="144.78" size="1.778" layer="91">Seram utilizados os pinos 34 e 35 para os Octocopladores, utilizaremos a conexão de jst de optocopladores dessa placa para isso.</text>
+<text x="38.1" y="139.7" size="1.778" layer="91">Será utilizado as conexões seriais, dessa placa</text>
+<text x="38.1" y="134.62" size="1.778" layer="91">Utilizaremos o conector de GND e Bateria dessa placa</text>
 </plain>
 <instances>
