File: Placa de acionamento/Esquema Acionamento 01/Esquema 01 guilherme.sch (EAGLE design)
At the start: 22 parts, among them Q1 IRF540, Q2 IRF540, Q3 IRF540

Commit message: Add files via upload
Parts:
- added SKIB3: (no value), SparkFun-Connectors:CONN_022.54MM_SCREWTERM
Connections:
- net SKIB2_CONECTOR: now also SKIB3.1
- net VCC: now also SKIB3.2
Other:
- moved on the sheet: SKIB2
Changed lines of the file:
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@@
 <part name="SKIB1" library="SparkFun-Connectors" deviceset="CONN_02" device="2.54MM_SCREWTERM"/>
 <part name="SKIB2" library="SparkFun-Connectors" deviceset="CONN_02" device="2.54MM_SCREWTERM"/>
+<part name="P+4" library="supply1" library_urn="urn:adsk.eagle:library:371" deviceset="VCC" device=""/>
+<part name="SKIB3" library="SparkFun-Connectors" deviceset="CONN_02" device="2.54MM_SCREWTERM"/>
 </parts>
 <sheets>
@@
 <attribute name="VALUE" x="66.04" y="0" size="1.778" layer="96"/>
 </instance>
-<instance part="P+2" gate="VCC" x="68.58" y="38.1" smashed="yes">
-<attribute name="VALUE" x="66.04" y="35.56" size="1.778" layer="96" rot="R90"/>
+<instance part="P+2" gate="VCC" x="35.56" y="40.64" smashed="yes">
+<attribute name="VALUE" x="33.02" y="38.1" size="1.778" layer="96" rot="R90"/>
 </instance>
 <instance part="Q3" gate="G$1" x="60.96" y="-55.88" smashed="yes">
@@
 <attribute name="NAME" x="43.18" y="86.868" size="1.778" layer="95" font="vector"/>
 </instance>
-<instance part="SKIB2" gate="G$1" x="45.72" y="25.4" smashed="yes">
-<attribute name="VALUE" x="43.18" y="20.574" size="1.778" layer="96" font="vector"/>
-<attribute name="NAME" x="43.18" y="30.988" size="1.778" layer="95" font="vector"/>
+<instance part="SKIB2" gate="G$1" x="27.94" y="25.4" smashed="yes">
+<attribute name="VALUE" x="25.4" y="20.574" size="1.778" layer="96" font="vector"/>
+<attribute name="NAME" x="25.4" y="30.988" size="1.778" layer="95" font="vector"/>
+</instance>
+<instance part="P+4" gate="VCC" x="68.58" y="45.72" smashed="yes">
+<attribute name="VALUE" x="66.04" y="43.18" size="1.778" layer="96" rot="R90"/>
+</instance>
+<instance part="SKIB3" gate="G$1" x="45.72" y="33.02" smashed="yes">
+<attribute name="VALUE" x="43.18" y="28.194" size="1.778" layer="96" font="vector"/>
+<attribute name="NAME" x="43.18" y="38.608" size="1.778" layer="95" font="vector"/>
 </instance>
 </instances>
@@
 </segment>
 <segment>
-<pinref part="P+2" gate="VCC" pin="VCC"/>
-<wire x1="68.58" y1="35.56" x2="68.58" y2="30.48" width="0.1524" layer="91"/>
-<wire x1="53.34" y1="27.94" x2="58.42" y2="27.94" width="0.1524" layer="91"/>
-<wire x1="58.42" y1="27.94" x2="58.42" y2="30.48" width="0.1524" layer="91"/>
-<wire x1="58.42" y1="30.48" x2="68.58" y2="30.48" width="0.1524" layer="91"/>
-<label x="58.42" y="30.48" size="1.778" layer="95"/>
-<pinref part="SKIB2" gate="G$1" pin="2"/>
-</segment>
-<segment>
 <pinref part="SP" gate="G$1" pin="2"/>
 <wire x1="66.04" y1="-22.86" x2="66.04" y2="-27.94" width="0.1524" layer="91"/>
 <label x="66.04" y="-22.86" size="1.778" layer="95"/>
+</segment>
+<segment>
+<pinref part="P+2" gate="VCC" pin="VCC"/>
+<wire x1="35.56" y1="38.1" x2="35.56" y2="27.94" width="0.1524" layer="91"/>
+<pinref part="SKIB2" gate="G$1" pin="2"/>
+</segment>
+<segment>
+<pinref part="P+4" gate="VCC" pin="VCC"/>
+<wire x1="68.58" y1="43.18" x2="68.58" y2="38.1" width="0.1524" layer="91"/>
+<wire x1="53.34" y1="35.56" x2="58.42" y2="35.56" width="0.1524" layer="91"/>
+<wire x1="58.42" y1="35.56" x2="58.42" y2="38.1" width="0.1524" layer="91"/>
+<wire x1="58.42" y1="38.1" x2="68.58" y2="38.1" width="0.1524" layer="91"/>
+<label x="58.42" y="38.1" size="1.778" layer="95"/>
+<pinref part="SKIB3" gate="G$1" pin="2"/>
 </segment>
 </net>
@@
 </segment>
 <segment>
+<wire x1="68.58" y1="20.32" x2="68.58" y2="27.94" width="0.1524" layer="91"/>
+<wire x1="58.42" y1="27.94" x2="68.58" y2="27.94" width="0.1524" layer="91"/>
+<wire x1="53.34" y1="33.02" x2="58.42" y2="33.02" width="0.1524" layer="91"/>
+<wire x1="58.42" y1="33.02" x2="58.42" y2="27.94" width="0.1524" layer="91"/>
+<label x="58.42" y="27.94" size="1.778" layer="95"/>
+<pinref part="SKIB3" gate="G$1" pin="1"/>
 <wire x1="68.58" y1="15.24" x2="68.58" y2="20.32" width="0.1524" layer="91"/>
-<wire x1="58.42" y1="20.32" x2="68.58" y2="20.32" width="0.1524" layer="91"/>
-<wire x1="53.34" y1="25.4" x2="58.42" y2="25.4" width="0.1524" layer="91"/>
-<wire x1="58.42" y1="25.4" x2="58.42" y2="20.32" width="0.1524" layer="91"/>
 <label x="58.42" y="20.32" size="1.778" layer="95"/>
 <pinref part="Q2" gate="G$1" pin="D"/>
 <pinref part="SKIB2" gate="G$1" pin="1"/>
-</segment>
-</net>
+<wire x1="68.58" y1="20.32" x2="35.56" y2="20.32" width="0.1524" layer="91"/>
+<wire x1="35.56" y1="20.32" x2="35.56" y2="25.4" width="0.1524" layer="91"/>
+<junction x="68.58" y="20.32"/>
+</segment>
+</net>
