File: Placa de processamento/Versões/Versão 1/Placa de processamento.brd (EAGLE design)
At the start: 90.2 x 100 mm, 12 parts

Commit message: Supostamente final com os modelos 3d corretos
Parts:
- removed U$1: PRESSION_BUTTON, CRD:PRESSION_BUTTON_FOOTPRINT
- added U$11: CHAVE_SS-5GL, CRD:CHAVESS-5GL
- moved SP1 2.54 mm to (10.2, 64.8)
- moved IC1 1.27 mm to (10.2, 38.1)
Connections:
- net VIN: now also U$11.P$2; no longer U$1.PL2, U$1.PR2
- net V_BATTERY: now also U$11.P$1; no longer U$1.PL1, U$1.PR1
Routing:
- net VIN: track 263.7 -> 505.3 mm
- net V_BATTERY: track 95.5 -> 54.1 mm
- net 5V: track 46.9 -> 45.6 mm
- net SKIB2: track 78.7 -> 79.9 mm
- net BUZZER: track 57.4 -> 58.6 mm
