File: Placa de processamento/Versões/Versão 1/Placa de processamento.sch (EAGLE design)
At the start: 12 parts

Commit message: Supostamente final com os modelos 3d corretos
Parts:
- removed U$1: PRESSION_BUTTON, CRD:PRESSION_BUTTON
- added U$11: CHAVE_SS-5GL, CRD:CHAVE_SS-5GL
Connections:
- net VIN: now also U$11.P$2; no longer U$1.PL2, U$1.PR2
- net V_BATTERY: now also U$11.P$1; no longer U$1.PL1, U$1.PR1
Changed lines of the file:
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@@
 <drawing>
 <settings>
-<setting alwaysvectorfont="yes"/>
+<setting alwaysvectorfont="no"/>
 <setting verticaltext="up"/>
 </settings>
@@
 </classes>
 <parts>
-<part name="U$1" library="CRD" library_urn="urn:adsk.eagle:library:39051337" deviceset="PRESSION_BUTTON" device="" package3d_urn="urn:adsk.eagle:package:43483815/3"/>
-<part name="U$2" library="CRD" library_urn="urn:adsk.eagle:library:39051337" deviceset="MICROSD_SMALL_READER" device="" package3d_urn="urn:adsk.eagle:package:44017969/2"/>
+<part name="U$2" library="CRD" library_urn="urn:adsk.eagle:library:39051337" deviceset="MICROSD_SMALL_READER" device="" package3d_urn="urn:adsk.eagle:package:44017969/2" override_package3d_urn="urn:adsk.eagle:package:44017969/3" override_package_urn="urn:adsk.eagle:footprint:44017967/2"/>
 <part name="U$3" library="CRD" library_urn="urn:adsk.eagle:library:39051337" deviceset="JST2.54X2P" device="" package3d_urn="urn:adsk.eagle:package:39191967/2"/>
 <part name="U$4" library="CRD" library_urn="urn:adsk.eagle:library:39051337" deviceset="JST2.54X2P" device="" package3d_urn="urn:adsk.eagle:package:39191967/2"/>
 <part name="U$5" library="CRD" library_urn="urn:adsk.eagle:library:39051337" deviceset="JST2.54X2P" device="" package3d_urn="urn:adsk.eagle:package:39191967/2"/>
 <part name="U$6" library="CRD" library_urn="urn:adsk.eagle:library:39051337" deviceset="JST2.54X2P" device="" package3d_urn="urn:adsk.eagle:package:39191967/2"/>
-<part name="U$7" library="CRD" library_urn="urn:adsk.eagle:library:39051337" deviceset="GPS_MODULE" device="" package3d_urn="urn:adsk.eagle:package:39608400/5"/>
-<part name="U$8" library="CRD" library_urn="urn:adsk.eagle:library:39051337" deviceset="E22-400T30D" device="" package3d_urn="urn:adsk.eagle:package:40965099/4"/>
-<part name="U$9" library="ESP32-DEVKITV1" library_urn="urn:adsk.eagle:library:44018017" deviceset="ESP32DEVKITV1" device="" package3d_urn="urn:adsk.eagle:package:44018021/1"/>
-<part name="IC1" library="v-reg" library_urn="urn:adsk.eagle:library:409" deviceset="78XXL" device="" package3d_urn="urn:adsk.eagle:package:30361/1"/>
+<part name="U$7" library="CRD" library_urn="urn:adsk.eagle:library:39051337" deviceset="GPS_MODULE" device="" package3d_urn="urn:adsk.eagle:package:39608400/5" override_package3d_urn="urn:adsk.eagle:package:49474690/2" override_package_urn="urn:adsk.eagle:footprint:39608398/5"/>
+<part name="U$8" library="CRD" library_urn="urn:adsk.eagle:library:39051337" deviceset="E22-400T30D" device="" package3d_urn="urn:adsk.eagle:package:40965099/4" override_package3d_urn="urn:adsk.eagle:package:40965099/7" override_package_urn="urn:adsk.eagle:footprint:40965097/4"/>
+<part name="U$9" library="ESP32-DEVKITV1" library_urn="urn:adsk.eagle:library:44018017" deviceset="ESP32DEVKITV1" device="" package3d_urn="urn:adsk.eagle:package:44018021/1" override_package3d_urn="urn:adsk.eagle:package:44018021/5" override_package_urn="urn:adsk.eagle:footprint:44018019/1"/>
+<part name="IC1" library="v-reg" library_urn="urn:adsk.eagle:library:409" deviceset="78XXL" device="" package3d_urn="urn:adsk.eagle:package:30361/1" override_package3d_urn="urn:adsk.eagle:package:49481284/2" override_package_urn="urn:adsk.eagle:footprint:30303/1"/>
 <part name="U$10" library="CRD" library_urn="urn:adsk.eagle:library:39051337" deviceset="JST2.54X2P" device="" package3d_urn="urn:adsk.eagle:package:39191967/2"/>
-<part name="SP1" library="buzzer" library_urn="urn:adsk.eagle:library:113" deviceset="AL11P" device="" package3d_urn="urn:adsk.eagle:package:5308/1"/>
+<part name="SP1" library="buzzer" library_urn="urn:adsk.eagle:library:113" deviceset="AL11P" device="" package3d_urn="urn:adsk.eagle:package:5308/1" override_package3d_urn="urn:adsk.eagle:package:49474686/2" override_package_urn="urn:adsk.eagle:footprint:5250/1"/>
+<part name="U$11" library="CRD" library_urn="urn:adsk.eagle:library:39051337" deviceset="CHAVE_SS-5GL" device="" package3d_urn="urn:adsk.eagle:package:45208058/14"/>
 </parts>
 <sheets>
@@
 </plain>
 <instances>
-<instance part="U$1" gate="G$1" x="17.78" y="71.12" smashed="yes"/>
 <instance part="U$2" gate="G$1" x="-35.56" y="7.62" smashed="yes"/>
 <instance part="U$3" gate="G$1" x="45.72" y="119.38" smashed="yes"/>
@@
 <attribute name="VALUE" x="176.53" y="111.125" size="1.778" layer="96"/>
 </instance>
+<instance part="U$11" gate="G$1" x="-45.72" y="73.66" smashed="yes"/>
 </instances>
 <busses>
@@
 </segment>
 <segment>
-<pinref part="U$1" gate="G$1" pin="PL1"/>
-<wire x1="6.35" y1="58.42" x2="6.35" y2="48.26" width="0.1524" layer="91"/>
-<wire x1="6.35" y1="48.26" x2="7.62" y2="48.26" width="0.1524" layer="91"/>
-<label x="5.08" y="43.18" size="1.778" layer="95" rot="R90"/>
-</segment>
-<segment>
-<pinref part="U$1" gate="G$1" pin="PR1"/>
-<wire x1="6.35" y1="83.82" x2="6.35" y2="93.98" width="0.1524" layer="91"/>
-<wire x1="6.35" y1="93.98" x2="7.62" y2="93.98" width="0.1524" layer="91"/>
-<label x="5.08" y="88.9" size="1.778" layer="95" rot="R90"/>
+<pinref part="U$11" gate="G$1" pin="P$1"/>
+<wire x1="-55.88" y1="60.96" x2="-55.88" y2="48.26" width="0.1524" layer="91"/>
+<wire x1="-55.88" y1="48.26" x2="-53.34" y2="48.26" width="0.1524" layer="91"/>
+<label x="-55.88" y="43.18" size="1.778" layer="95" rot="R90"/>
 </segment>
 </net>
@@
 </segment>
 <segment>
-<pinref part="U$1" gate="G$1" pin="PL2"/>
-<wire x1="11.43" y1="58.42" x2="11.43" y2="48.26" width="0.1524" layer="91"/>
-<wire x1="11.43" y1="48.26" x2="12.7" y2="48.26" width="0.1524" layer="91"/>
-<label x="9.398" y="55.118" size="1.778" layer="95" rot="R270"/>
-</segment>
-<segment>
-<pinref part="U$1" gate="G$1" pin="PR2"/>
-<wire x1="11.43" y1="83.82" x2="11.43" y2="93.98" width="0.1524" layer="91"/>
-<wire x1="11.43" y1="93.98" x2="12.7" y2="93.98" width="0.1524" layer="91"/>
-<label x="11.176" y="87.122" size="1.778" layer="95" rot="R90"/>
+<pinref part="U$11" gate="G$1" pin="P$2"/>
+<wire x1="-45.72" y1="60.96" x2="-45.72" y2="48.26" width="0.1524" layer="91"/>
+<wire x1="-45.72" y1="48.26" x2="-43.18" y2="48.26" width="0.1524" layer="91"/>
+<label x="-45.72" y="53.34" size="1.778" layer="95" rot="R90"/>
 </segment>
 </net>
@@
 packages will not be understood (or retained) with this version.
 </note>
+<note version="9.4" severity="warning">
+Since Version 9.4, EAGLE supports the overriding of 3D packages
+in schematics and board files. Those overridden 3d packages
+will not be understood (or retained) with this version.
+</note>
 </compatibility>
