File: COTS/Versões/Versão 1/COTS.brd (EAGLE design)
At the start: 76.2 x 79.7 mm, 10 parts

Commit message: Supostamente final com os modelos 3d corretos
Parts:
- removed U$10: PRESSION_BUTTON, CRD:PRESSION_BUTTON_FOOTPRINT
- added IC1: (no value), v-reg:78XXL
- added U$8: CHAVE_SS-5GL, CRD:CHAVESS-5GL
- moved SP2 6.48 mm to (11.9, 54.4)
- moved U$1 4.02 mm to (16.5, 16.5)
- moved U$3 4.02 mm to (16.5, 33.0)
- moved U$4 2.54 mm to (45.7, 66.0)
- moved U$9 2.54 mm to (36.8, 66.0)
- moved U$5 2.54 mm to (45.7, 73.7)
- moved U$6 2.54 mm to (36.8, 73.7)
- moved U$7 2.54 mm to (54.6, 69.8)
Connections:
- new net 5V: IC1.OUT, U$2.30
- net GND: now also IC1.GND
- net VIN: now also IC1.IN, U$8.P$1; no longer U$10.PL1, U$10.PR1, U$2.30
- net V_BATTERY: now also U$8.P$2; no longer U$10.PL2, U$10.PR2
Routing:
- net VIN: track 98.2 -> 37.8 mm
- net 5V: track 0.00 -> 35.5 mm, vias 0 -> 2
- net BUZZER: track 41.9 -> 47.4 mm
- net SCL: track 130.9 -> 135.2 mm
- net 3V3: track 179.7 -> 176.9 mm
- net V_BATTERY: track 25.0 -> 27.6 mm
- net SKIB2: track 48.4 -> 50.9 mm
- net SKIB1: track 52.0 -> 54.6 mm
- net OPTOACOPLADOR2: track 27.8 -> 30.4 mm
- net OPTOACOPLADOR1: track 24.0 -> 26.5 mm
- net SIGNAL1: track 48.0 -> 50.5 mm
- net TX2: track 51.2 -> 53.7 mm
- net RX2: track 54.9 -> 56.0 mm
- net SDA: track 98.9 -> 98.2 mm
- added copper zone on layer 1, net GND

Commit message: Atualizando plata COTS
Parts:
- added U$10: BMP280V1, CRD:BMP280_FOOTPRINT
- moved IC1 4.02 mm to (25.4, 52.1)
- moved U$3 3.81 mm to (16.5, 36.8)
- moved U$1 1.80 mm to (17.8, 15.2), turned to 270 degrees
- moved U$4 1.27 mm to (45.7, 64.8)
- moved U$9 1.27 mm to (36.8, 64.8)
- moved U$8 1.27 mm to (19.1, 72.4)
- renumbered SP2 to SP1
Connections:
- net 3V3: now also U$10.VCC
- net GND: now also U$10.GND; no longer U$2.2
- net SCL: now also U$10.SCL
- net SDA: now also U$10.SDA
- net V_BATTERY: now also U$8.P$3; no longer U$8.P$2
Routing:
- net SDA: track 98.2 -> 126.1 mm
- net 3V3: track 176.9 -> 204.1 mm
- net SCL: track 135.2 -> 158.7 mm
- net V_BATTERY: track 27.6 -> 9.48 mm
- net VIN: track 37.8 -> 32.6 mm
- net 5V: track 35.5 -> 40.6 mm
- net GND: track 2.29 -> 6.73 mm, vias 0 -> 2
- net SKIB2: track 50.9 -> 48.5 mm
- net OPTOACOPLADOR2: track 30.4 -> 32.7 mm
- net TX2: track 53.7 -> 51.7 mm
- net RX2: track 56.0 -> 56.7 mm
- net BUZZER: track 47.4 -> 46.7 mm
- net SKIB1: track 54.6 -> 54.0 mm
- net OPTOACOPLADOR1: track 26.5 -> 27.0 mm
- removed copper zone on layer 1, net GND
