File: COTS/Versões/Versão 1/COTS.sch (EAGLE design)
At the start: 10 parts

Commit message: Supostamente final com os modelos 3d corretos
Parts:
- removed U$10: PRESSION_BUTTON, CRD:PRESSION_BUTTON
- added IC1: (no value), v-reg:78XXL
- added U$8: CHAVE_SS-5GL, CRD:CHAVE_SS-5GL
Connections:
- new net 5V: IC1.OUT, U$2.VIN
- net GND: now also IC1.GND
- net VIN: now also IC1.IN, U$8.P$1; no longer U$10.PL1, U$10.PR1, U$2.VIN
- net V_BATTERY: now also U$8.P$2; no longer U$10.PL2, U$10.PR2
Changed lines of the file:
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@@
 <drawing>
 <settings>
-<setting alwaysvectorfont="yes"/>
+<setting alwaysvectorfont="no"/>
 <setting verticaltext="up"/>
 </settings>
@@
 </classes>
 <parts>
-<part name="U$1" library="CRD" library_urn="urn:adsk.eagle:library:39051337" deviceset="MPU6050" device="V1" package3d_urn="urn:adsk.eagle:package:39029071/8"/>
-<part name="U$2" library="ESP32-DEVKITV1" library_urn="urn:adsk.eagle:library:44018017" deviceset="ESP32DEVKITV1" device="" package3d_urn="urn:adsk.eagle:package:44018021/1"/>
-<part name="U$3" library="CRD" library_urn="urn:adsk.eagle:library:39051337" deviceset="BMP390" device="V1" package3d_urn="urn:adsk.eagle:package:40965124/5"/>
-<part name="U$4" library="CRD" library_urn="urn:adsk.eagle:library:39051337" deviceset="JST2.54X2P" device="" package3d_urn="urn:adsk.eagle:package:39191967/2"/>
+<part name="U$1" library="CRD" library_urn="urn:adsk.eagle:library:39051337" deviceset="MPU6050" device="V1" package3d_urn="urn:adsk.eagle:package:39029071/8" override_package3d_urn="urn:adsk.eagle:package:49473311/2" override_package_urn="urn:adsk.eagle:footprint:39029067/6"/>
+<part name="U$2" library="ESP32-DEVKITV1" library_urn="urn:adsk.eagle:library:44018017" deviceset="ESP32DEVKITV1" device="" package3d_urn="urn:adsk.eagle:package:44018021/1" override_package3d_urn="urn:adsk.eagle:package:44018021/2" override_package_urn="urn:adsk.eagle:footprint:44018019/1"/>
+<part name="U$3" library="CRD" library_urn="urn:adsk.eagle:library:39051337" deviceset="BMP390" device="V1" package3d_urn="urn:adsk.eagle:package:40965124/5" override_package3d_urn="urn:adsk.eagle:package:49473309/2" override_package_urn="urn:adsk.eagle:footprint:40965120/5"/>
+<part name="U$4" library="CRD" library_urn="urn:adsk.eagle:library:39051337" deviceset="JST2.54X2P" device="" package3d_urn="urn:adsk.eagle:package:39191967/2" override_package3d_urn="urn:adsk.eagle:package:49473313/2" override_package_urn="urn:adsk.eagle:footprint:39191965/1"/>
 <part name="U$5" library="CRD" library_urn="urn:adsk.eagle:library:39051337" deviceset="JST2.54X2P" device="" package3d_urn="urn:adsk.eagle:package:39191967/2"/>
 <part name="U$6" library="CRD" library_urn="urn:adsk.eagle:library:39051337" deviceset="JST2.54X2P" device="" package3d_urn="urn:adsk.eagle:package:39191967/2"/>
 <part name="U$7" library="CRD" library_urn="urn:adsk.eagle:library:39051337" deviceset="JST2.54X2P" device="" package3d_urn="urn:adsk.eagle:package:39191967/2"/>
 <part name="U$9" library="CRD" library_urn="urn:adsk.eagle:library:39051337" deviceset="JST2.54X2P" device="" package3d_urn="urn:adsk.eagle:package:39191967/2"/>
-<part name="U$10" library="CRD" library_urn="urn:adsk.eagle:library:39051337" deviceset="PRESSION_BUTTON" device="" package3d_urn="urn:adsk.eagle:package:43483815/3"/>
-<part name="SP2" library="buzzer" library_urn="urn:adsk.eagle:library:113" deviceset="AL11P" device="" package3d_urn="urn:adsk.eagle:package:5308/1"/>
+<part name="SP2" library="buzzer" library_urn="urn:adsk.eagle:library:113" deviceset="AL11P" device="" package3d_urn="urn:adsk.eagle:package:5308/1" override_package3d_urn="urn:adsk.eagle:package:49481862/2" override_package_urn="urn:adsk.eagle:footprint:5250/1"/>
+<part name="IC1" library="v-reg" library_urn="urn:adsk.eagle:library:409" deviceset="78XXL" device="" package3d_urn="urn:adsk.eagle:package:30361/1" override_package3d_urn="urn:adsk.eagle:package:49481863/2" override_package_urn="urn:adsk.eagle:footprint:30303/1"/>
+<part name="U$8" library="CRD" library_urn="urn:adsk.eagle:library:39051337" deviceset="CHAVE_SS-5GL" device="" package3d_urn="urn:adsk.eagle:package:45208058/14"/>
 </parts>
 <sheets>
@@
 <instance part="U$7" gate="G$1" x="60.96" y="116.84" smashed="yes"/>
 <instance part="U$9" gate="G$1" x="-73.66" y="116.84" smashed="yes"/>
-<instance part="U$10" gate="G$1" x="195.58" y="58.42" smashed="yes"/>
 <instance part="SP2" gate="G$1" x="236.22" y="53.34" smashed="yes">
 <attribute name="NAME" x="232.41" y="59.69" size="1.778" layer="95"/>
 <attribute name="VALUE" x="232.41" y="50.165" size="1.778" layer="96"/>
 </instance>
+<instance part="IC1" gate="A" x="-35.56" y="68.58" smashed="yes">
+<attribute name="NAME" x="-33.02" y="60.96" size="1.778" layer="95"/>
+<attribute name="VALUE" x="-33.02" y="58.42" size="1.778" layer="96"/>
+</instance>
+<instance part="U$8" gate="G$1" x="236.22" y="101.6" smashed="yes"/>
 </instances>
 <busses>
@@
 <net name="VIN" class="0">
 <segment>
-<pinref part="U$2" gate="G$1" pin="VIN"/>
-<wire x1="83.82" y1="30.48" x2="73.66" y2="30.48" width="0.1524" layer="91"/>
-<label x="73.66" y="30.48" size="1.778" layer="95"/>
-</segment>
-<segment>
 <wire x1="154.94" y1="50.8" x2="154.94" y2="43.18" width="0.1524" layer="91"/>
 <label x="154.94" y="38.1" size="1.778" layer="95" rot="R90"/>
@@
 </segment>
 <segment>
-<pinref part="U$10" gate="G$1" pin="PL1"/>
-<wire x1="184.15" y1="45.72" x2="184.15" y2="38.1" width="0.1524" layer="91"/>
-<wire x1="184.15" y1="38.1" x2="182.88" y2="38.1" width="0.1524" layer="91"/>
-<label x="182.88" y="33.02" size="1.778" layer="95" rot="R90"/>
-</segment>
-<segment>
-<pinref part="U$10" gate="G$1" pin="PR1"/>
-<wire x1="184.15" y1="71.12" x2="184.15" y2="78.74" width="0.1524" layer="91"/>
-<wire x1="184.15" y1="78.74" x2="182.88" y2="78.74" width="0.1524" layer="91"/>
-<label x="182.88" y="78.74" size="1.778" layer="95" rot="R90"/>
+<pinref part="IC1" gate="A" pin="IN"/>
+<wire x1="-43.18" y1="68.58" x2="-48.26" y2="68.58" width="0.1524" layer="91"/>
+<label x="-50.8" y="68.58" size="1.778" layer="95"/>
+</segment>
+<segment>
+<pinref part="U$8" gate="G$1" pin="P$1"/>
+<wire x1="226.06" y1="88.9" x2="226.06" y2="78.74" width="0.1524" layer="91"/>
+<wire x1="226.06" y1="78.74" x2="223.52" y2="78.74" width="0.1524" layer="91"/>
+<label x="220.98" y="78.74" size="1.778" layer="95" rot="R90"/>
 </segment>
 </net>
@@
 <label x="228.6" y="43.18" size="1.778" layer="95"/>
 </segment>
+<segment>
+<pinref part="IC1" gate="A" pin="GND"/>
+<wire x1="-35.56" y1="60.96" x2="-35.56" y2="55.88" width="0.1524" layer="91"/>
+<label x="-35.56" y="53.34" size="1.778" layer="95"/>
+</segment>
 </net>
 <net name="SKIB1" class="0">
@@
 </segment>
 <segment>
-<pinref part="U$10" gate="G$1" pin="PL2"/>
-<wire x1="189.23" y1="45.72" x2="189.23" y2="38.1" width="0.1524" layer="91"/>
-<wire x1="189.23" y1="38.1" x2="187.96" y2="38.1" width="0.1524" layer="91"/>
-<label x="187.96" y="27.94" size="1.778" layer="95" rot="R90"/>
-</segment>
-<segment>
-<pinref part="U$10" gate="G$1" pin="PR2"/>
-<wire x1="189.23" y1="71.12" x2="189.23" y2="78.74" width="0.1524" layer="91"/>
-<wire x1="189.23" y1="78.74" x2="187.96" y2="78.74" width="0.1524" layer="91"/>
-<label x="187.96" y="76.2" size="1.778" layer="95" rot="R90"/>
+<pinref part="U$8" gate="G$1" pin="P$2"/>
+<wire x1="236.22" y1="88.9" x2="236.22" y2="78.74" width="0.1524" layer="91"/>
+<wire x1="236.22" y1="78.74" x2="233.68" y2="78.74" width="0.1524" layer="91"/>
+<label x="231.14" y="76.2" size="1.778" layer="95" rot="R90"/>
 </segment>
 </net>
@@
 <wire x1="83.82" y1="43.18" x2="73.66" y2="43.18" width="0.1524" layer="91"/>
 <label x="73.66" y="43.18" size="1.778" layer="95"/>
+</segment>
+</net>
+<net name="5V" class="0">
+<segment>
+<pinref part="IC1" gate="A" pin="OUT"/>
+<wire x1="-27.94" y1="68.58" x2="-22.86" y2="68.58" width="0.1524" layer="91"/>
+<label x="-22.86" y="68.58" size="1.778" layer="95"/>
+</segment>
+<segment>
+<pinref part="U$2" gate="G$1" pin="VIN"/>
+<wire x1="83.82" y1="30.48" x2="73.66" y2="30.48" width="0.1524" layer="91"/>
+<label x="73.66" y="30.48" size="1.778" layer="95"/>
 </segment>
 </net>
@@
 packages will not be understood (or retained) with this version.
 </note>
+<note version="9.4" severity="warning">
+Since Version 9.4, EAGLE supports the overriding of 3D packages
+in schematics and board files. Those overridden 3d packages
+will not be understood (or retained) with this version.
+</note>
 </compatibility>

Commit message: Atualizando plata COTS
Parts:
- removed SP2: AL11P, buzzer:AL11P
- added SP1: AL11P, buzzer:AL11P
- added U$10: BMP280V1, CRD:BMP280V1
Connections:
- net 3V3: now also U$10.VCC
- net BUZZER: now also SP1.2; no longer SP2.2
- net GND: now also SP1.1, U$10.GND; no longer SP2.1, U$2.GND
- net SCL: now also U$10.SCL
- net SDA: now also U$10.SDA
- net V_BATTERY: now also U$8.P$3; no longer U$8.P$2
Changed lines of the file:
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@@
 </classes>
 <parts>
-<part name="U$1" library="CRD" library_urn="urn:adsk.eagle:library:39051337" deviceset="MPU6050" device="V1" package3d_urn="urn:adsk.eagle:package:39029071/8" override_package3d_urn="urn:adsk.eagle:package:49473311/2" override_package_urn="urn:adsk.eagle:footprint:39029067/6"/>
-<part name="U$2" library="ESP32-DEVKITV1" library_urn="urn:adsk.eagle:library:44018017" deviceset="ESP32DEVKITV1" device="" package3d_urn="urn:adsk.eagle:package:44018021/1" override_package3d_urn="urn:adsk.eagle:package:44018021/2" override_package_urn="urn:adsk.eagle:footprint:44018019/1"/>
-<part name="U$3" library="CRD" library_urn="urn:adsk.eagle:library:39051337" deviceset="BMP390" device="V1" package3d_urn="urn:adsk.eagle:package:40965124/5" override_package3d_urn="urn:adsk.eagle:package:49473309/2" override_package_urn="urn:adsk.eagle:footprint:40965120/5"/>
-<part name="U$4" library="CRD" library_urn="urn:adsk.eagle:library:39051337" deviceset="JST2.54X2P" device="" package3d_urn="urn:adsk.eagle:package:39191967/2" override_package3d_urn="urn:adsk.eagle:package:49473313/2" override_package_urn="urn:adsk.eagle:footprint:39191965/1"/>
-<part name="U$5" library="CRD" library_urn="urn:adsk.eagle:library:39051337" deviceset="JST2.54X2P" device="" package3d_urn="urn:adsk.eagle:package:39191967/2"/>
-<part name="U$6" library="CRD" library_urn="urn:adsk.eagle:library:39051337" deviceset="JST2.54X2P" device="" package3d_urn="urn:adsk.eagle:package:39191967/2"/>
-<part name="U$7" library="CRD" library_urn="urn:adsk.eagle:library:39051337" deviceset="JST2.54X2P" device="" package3d_urn="urn:adsk.eagle:package:39191967/2"/>
-<part name="U$9" library="CRD" library_urn="urn:adsk.eagle:library:39051337" deviceset="JST2.54X2P" device="" package3d_urn="urn:adsk.eagle:package:39191967/2"/>
-<part name="SP2" library="buzzer" library_urn="urn:adsk.eagle:library:113" deviceset="AL11P" device="" package3d_urn="urn:adsk.eagle:package:5308/1" override_package3d_urn="urn:adsk.eagle:package:49481862/2" override_package_urn="urn:adsk.eagle:footprint:5250/1"/>
+<part name="U$1" library="CRD" library_urn="urn:adsk.eagle:library:39051337" deviceset="MPU6050" device="V1" package3d_urn="urn:adsk.eagle:package:39029071/10" override_package3d_urn="urn:adsk.eagle:package:49473311/2" override_package_urn="urn:adsk.eagle:footprint:39029067/6" override_locally_modified="yes"/>
+<part name="U$2" library="ESP32-DEVKITV1" library_urn="urn:adsk.eagle:library:44018017" deviceset="ESP32DEVKITV1" device="" package3d_urn="urn:adsk.eagle:package:44018021/2" override_package3d_urn="urn:adsk.eagle:package:49887807/2" override_package_urn="urn:adsk.eagle:footprint:49887808/1"/>
+<part name="U$3" library="CRD" library_urn="urn:adsk.eagle:library:39051337" deviceset="BMP390" device="V1" package3d_urn="urn:adsk.eagle:package:40965124/8" override_package3d_urn="urn:adsk.eagle:package:49473309/2" override_package_urn="urn:adsk.eagle:footprint:40965120/5" override_locally_modified="yes"/>
+<part name="U$4" library="CRD" library_urn="urn:adsk.eagle:library:39051337" deviceset="JST2.54X2P" device="" package3d_urn="urn:adsk.eagle:package:39191967/3" override_package3d_urn="urn:adsk.eagle:package:49473313/2" override_package_urn="urn:adsk.eagle:footprint:39191965/1" override_locally_modified="yes"/>
+<part name="U$5" library="CRD" library_urn="urn:adsk.eagle:library:39051337" deviceset="JST2.54X2P" device="" package3d_urn="urn:adsk.eagle:package:39191967/3"/>
+<part name="U$6" library="CRD" library_urn="urn:adsk.eagle:library:39051337" deviceset="JST2.54X2P" device="" package3d_urn="urn:adsk.eagle:package:39191967/3"/>
+<part name="U$7" library="CRD" library_urn="urn:adsk.eagle:library:39051337" deviceset="JST2.54X2P" device="" package3d_urn="urn:adsk.eagle:package:39191967/3"/>
+<part name="U$9" library="CRD" library_urn="urn:adsk.eagle:library:39051337" deviceset="JST2.54X2P" device="" package3d_urn="urn:adsk.eagle:package:39191967/3"/>
 <part name="IC1" library="v-reg" library_urn="urn:adsk.eagle:library:409" deviceset="78XXL" device="" package3d_urn="urn:adsk.eagle:package:30361/1" override_package3d_urn="urn:adsk.eagle:package:49481863/2" override_package_urn="urn:adsk.eagle:footprint:30303/1"/>
 <part name="U$8" library="CRD" library_urn="urn:adsk.eagle:library:39051337" deviceset="CHAVE_SS-5GL" device="" package3d_urn="urn:adsk.eagle:package:45208058/14"/>
+<part name="U$10" library="CRD" library_urn="urn:adsk.eagle:library:39051337" deviceset="BMP280" device="V1" package3d_urn="urn:adsk.eagle:package:39029072/8" override_package3d_urn="urn:adsk.eagle:package:39029072/9" override_package_urn="urn:adsk.eagle:footprint:39029068/5"/>
+<part name="SP1" library="buzzer" deviceset="AL11P" device="" package3d_urn="urn:adsk.eagle:package:5308/1" override_package3d_urn="urn:adsk.eagle:package:49887804/2" override_package_urn="urn:adsk.eagle:footprint:49887805/1"/>
 </parts>
 <sheets>
@@
 <instance part="U$7" gate="G$1" x="60.96" y="116.84" smashed="yes"/>
 <instance part="U$9" gate="G$1" x="-73.66" y="116.84" smashed="yes"/>
-<instance part="SP2" gate="G$1" x="236.22" y="53.34" smashed="yes">
-<attribute name="NAME" x="232.41" y="59.69" size="1.778" layer="95"/>
-<attribute name="VALUE" x="232.41" y="50.165" size="1.778" layer="96"/>
-</instance>
 <instance part="IC1" gate="A" x="-35.56" y="68.58" smashed="yes">
 <attribute name="NAME" x="-33.02" y="60.96" size="1.778" layer="95"/>
@@
 </instance>
 <instance part="U$8" gate="G$1" x="236.22" y="101.6" smashed="yes"/>
+<instance part="U$10" gate="G$1" x="88.9" y="5.08" smashed="yes"/>
+<instance part="SP1" gate="G$1" x="236.22" y="48.26" smashed="yes">
+<attribute name="NAME" x="232.41" y="54.61" size="1.778" layer="95"/>
+<attribute name="VALUE" x="232.41" y="45.085" size="1.778" layer="96"/>
+</instance>
 </instances>
 <busses>
@@
 </segment>
 <segment>
-<pinref part="U$2" gate="G$1" pin="GND"/>
-<wire x1="119.38" y1="33.02" x2="129.54" y2="33.02" width="0.1524" layer="91"/>
-<label x="129.54" y="33.02" size="1.778" layer="95"/>
-</segment>
-<segment>
 <pinref part="U$1" gate="G$1" pin="GND"/>
 <wire x1="15.24" y1="40.64" x2="15.24" y2="33.02" width="0.1524" layer="91"/>
@@
 </segment>
 <segment>
-<pinref part="SP2" gate="G$1" pin="1"/>
-<wire x1="231.14" y1="53.34" x2="228.6" y2="53.34" width="0.1524" layer="91"/>
-<wire x1="228.6" y1="53.34" x2="228.6" y2="45.72" width="0.1524" layer="91"/>
-<label x="228.6" y="43.18" size="1.778" layer="95"/>
-</segment>
-<segment>
 <pinref part="IC1" gate="A" pin="GND"/>
 <wire x1="-35.56" y1="60.96" x2="-35.56" y2="55.88" width="0.1524" layer="91"/>
 <label x="-35.56" y="53.34" size="1.778" layer="95"/>
 </segment>
+<segment>
+<pinref part="U$10" gate="G$1" pin="GND"/>
+<wire x1="81.28" y1="-10.16" x2="81.28" y2="-17.78" width="0.1524" layer="91"/>
+<label x="81.28" y="-20.32" size="1.778" layer="95" rot="R90"/>
+</segment>
+<segment>
+<pinref part="SP1" gate="G$1" pin="1"/>
+<wire x1="231.14" y1="48.26" x2="228.6" y2="48.26" width="0.1524" layer="91"/>
+<wire x1="228.6" y1="48.26" x2="228.6" y2="38.1" width="0.1524" layer="91"/>
+<label x="228.6" y="35.56" size="1.778" layer="95"/>
+</segment>
 </net>
 <net name="SKIB1" class="0">
@@
 <net name="BUZZER" class="0">
 <segment>
-<pinref part="SP2" gate="G$1" pin="2"/>
-<wire x1="241.3" y1="53.34" x2="243.84" y2="53.34" width="0.1524" layer="91"/>
-<wire x1="243.84" y1="53.34" x2="243.84" y2="45.72" width="0.1524" layer="91"/>
-<label x="243.84" y="43.18" size="1.778" layer="95"/>
-</segment>
-<segment>
 <pinref part="U$2" gate="G$1" pin="IO14"/>
 <wire x1="83.82" y1="40.64" x2="73.66" y2="40.64" width="0.1524" layer="91"/>
 <label x="73.66" y="40.64" size="1.778" layer="95"/>
 </segment>
+<segment>
+<pinref part="SP1" gate="G$1" pin="2"/>
+<wire x1="241.3" y1="48.26" x2="243.84" y2="48.26" width="0.1524" layer="91"/>
+<wire x1="243.84" y1="48.26" x2="243.84" y2="38.1" width="0.1524" layer="91"/>
+<label x="243.84" y="35.56" size="1.778" layer="95"/>
+</segment>
 </net>
 <net name="SDA" class="0">
@@
 <label x="48.26" y="-12.7" size="1.778" layer="95" rot="R90"/>
 </segment>
+<segment>
+<pinref part="U$10" gate="G$1" pin="SDA"/>
+<wire x1="91.44" y1="-10.16" x2="91.44" y2="-17.78" width="0.1524" layer="91"/>
+<label x="91.44" y="-20.32" size="1.778" layer="95" rot="R90"/>
+</segment>
 </net>
 <net name="SCL" class="0">
@@
 <label x="38.1" y="-12.7" size="1.778" layer="95" rot="R90"/>
 </segment>
+<segment>
+<pinref part="U$10" gate="G$1" pin="SCL"/>
+<wire x1="86.36" y1="-10.16" x2="86.36" y2="-17.78" width="0.1524" layer="91"/>
+<label x="86.36" y="-20.32" size="1.778" layer="95" rot="R90"/>
+</segment>
 </net>
 <net name="3V3" class="0">
@@
 <label x="10.16" y="93.98" size="1.778" layer="95" rot="R90"/>
 </segment>
+<segment>
+<pinref part="U$10" gate="G$1" pin="VCC"/>
+<wire x1="76.2" y1="-10.16" x2="76.2" y2="-17.78" width="0.1524" layer="91"/>
+<label x="76.2" y="-20.32" size="1.778" layer="95" rot="R90"/>
+</segment>
 </net>
 <net name="V_BATTERY" class="0">
@@
 </segment>
 <segment>
-<pinref part="U$8" gate="G$1" pin="P$2"/>
-<wire x1="236.22" y1="88.9" x2="236.22" y2="78.74" width="0.1524" layer="91"/>
-<wire x1="236.22" y1="78.74" x2="233.68" y2="78.74" width="0.1524" layer="91"/>
-<label x="231.14" y="76.2" size="1.778" layer="95" rot="R90"/>
-</segment>
-</net>
+<pinref part="U$8" gate="G$1" pin="P$3"/>
+<wire x1="248.92" y1="88.9" x2="248.92" y2="78.74" width="0.1524" layer="91"/>
+<wire x1="248.92" y1="78.74" x2="246.38" y2="78.74" width="0.1524" layer="91"/>
+<label x="243.84" y="78.74" size="1.778" layer="95" rot="R90"/>
+</segment>
+</net>
